Commit message: Add visualize argument for the simulators

File: velodyne_description/urdf/HDL-32E.urdf.xacro (robot description, xacro)
@@ -2,5 +2,5 @@
 <robot xmlns:xacro="http://www.ros.org/wiki/xacro" name="HDL-32E">
   <xacro:property name="M_PI" value="3.1415926535897931" />
-  <xacro:macro name="HDL-32E" params="*origin parent:=base_link name:=velodyne topic:=/velodyne_points hz:=10 lasers:=32 samples:=2187 collision_range:=0.3 min_range:=0.9 max_range:=130.0 noise:=0.008 min_angle:=-${M_PI} max_angle:=${M_PI} gpu:=false">
+  <xacro:macro name="HDL-32E" params="*origin parent:=base_link name:=velodyne topic:=/velodyne_points hz:=10 lasers:=32 samples:=2187 collision_range:=0.3 min_range:=0.9 max_range:=130.0 noise:=0.008 min_angle:=-${M_PI} max_angle:=${M_PI} gpu:=false visualize:=false">
     <joint name="${name}_base_mount_joint" type="fixed">
       <xacro:insert_block name="origin" />
@@ -51,5 +51,5 @@
         <sensor type="gpu_ray" name="${name}-HDL32E">
           <pose>0 0 0 0 0 0</pose>
-          <visualize>false</visualize>
+          <visualize>${visualize}</visualize>
           <update_rate>${hz}</update_rate>
           <ray>
@@ -91,5 +91,5 @@
         <sensor type="ray" name="${name}-HDL32E">
           <pose>0 0 0 0 0 0</pose>
-          <visualize>false</visualize>
+          <visualize>${visualize}</visualize>
           <update_rate>${hz}</update_rate>
           <ray>

File: velodyne_description/urdf/VLP-16.urdf.xacro (robot description, xacro)
@@ -2,5 +2,5 @@
 <robot xmlns:xacro="http://www.ros.org/wiki/xacro" name="VLP-16">
   <xacro:property name="M_PI" value="3.1415926535897931" />
-  <xacro:macro name="VLP-16" params="*origin parent:=base_link name:=velodyne topic:=/velodyne_points hz:=10 lasers:=16 samples:=1875 collision_range:=0.3 min_range:=0.9 max_range:=130.0 noise:=0.008 min_angle:=-${M_PI} max_angle:=${M_PI} gpu:=false">
+  <xacro:macro name="VLP-16" params="*origin parent:=base_link name:=velodyne topic:=/velodyne_points hz:=10 lasers:=16 samples:=1875 collision_range:=0.3 min_range:=0.9 max_range:=130.0 noise:=0.008 min_angle:=-${M_PI} max_angle:=${M_PI} gpu:=false visualize:=false">
     <joint name="${name}_base_mount_joint" type="fixed">
       <xacro:insert_block name="origin" />
@@ -56,5 +56,5 @@
         <sensor type="gpu_ray" name="${name}-VLP16">
           <pose>0 0 0 0 0 0</pose>
-          <visualize>false</visualize>
+          <visualize>${visualize}</visualize>
           <update_rate>${hz}</update_rate>
           <ray>
@@ -96,5 +96,5 @@
         <sensor type="ray" name="${name}-VLP16">
           <pose>0 0 0 0 0 0</pose>
-          <visualize>false</visualize>
+          <visualize>${visualize}</visualize>
           <update_rate>${hz}</update_rate>
           <ray>
